File: Regular_PA_LNA/MySRaspiGW_PA_LNA.sch (KiCad schematic (older format))
At the start: 5 parts, among them P1 CONN_02X04, U1 NRF24L01

Commit message: v1.1 IRQ support
Added IRQ support on pin 18
Connections:
- net IRQ: now reaches U1.8 (IRQ)
- net IRQ: now also P1.2 (P2)
- no-connect marks 2 -> 0
Changed lines of the file:
@@
 LIBS:mysensors_security
 LIBS:mysensors_sensors
+LIBS:MySRaspiGW_PA_LNA-cache
 EELAYER 25 0
 EELAYER END
@@
 Sheet 1 1
 Title "MySRaspiGW"
-Date "05/29/2016"
-Rev "1.0"
+Date "03/13/2017"
+Rev "1.1"
 Comp "https://github.com/emc2cube/MySRaspiGW/tree/master/Regular"
 Comment1 ""
@@
 Connection ~ 4300 1050
 Connection ~ 4700 1050
-NoConn ~ 3750 1400
-NoConn ~ 1850 1200
 Wire Wire Line
 	1850 1300 2200 1300
+Text GLabel 1850 1200 2    60   Input ~ 0
+IRQ
+Text GLabel 3750 1400 2    60   Input ~ 0
+IRQ
 $EndSCHEMATC
